Commit message: Update widowx_turret.urdf.xacro
changes to work better with our current robot setup

File: widowx_turret_description/robots/widowx_turret.urdf.xacro (robot description, xacro)
@@ -10,6 +10,6 @@
 		</visual>
 	</link>
-	<xacro:widowx_turret parent="base_footprint" prefix="">
-		<origin xyz="0.0 0.0 0.0" rpy="0.0 0.0 0.0"/>
+	<xacro:widowx_turret parent="base_link" prefix="">
+		<origin xyz="0.0 0.0 0.0" rpy="0.0 0.0 -1.57"/>
 	</xacro:widowx_turret>
 </robot>
